Commit message: pcd_node: removed invalid distance data from pointclouds urdf: adjusted body size to correct height

File: urdfs/rc25.urdf (robot description, URDF)
Before this commit: robot rc25, 15 links, 14 joints
Links:
- link base_link: geometry visual box size=0.650 0.380 0.350; visual cylinder length=0.070 radius=0.090

Commit message: urdf: maybe camera, tof and lidar are aligned

File: urdfs/rc25.urdf (robot description, URDF)
Before this commit: robot rc25, 15 links, 14 joints
Joints:
- joint oak-d-base-frame: origin xyz=0.340 0.00 0.240 rpy=0 0 0.05 -> xyz=0.340 0.00 0.240 rpy=0.00 -0.05 0.00
