Commit message: rc.urdf: adjusted Lidar z rotation to align cone detec with camera

File: urdfs/rc.urdf (robot description, URDF)
Before this commit: robot rc, 15 links, 14 joints
Joints:
- joint lidar_joint: origin xyz=0.180 0 0.300 rpy=0 0 -0.025 -> xyz=0.180 0 0.300 rpy=0 0 -0.05

Commit message: .bashrc_rc: added more topics to rc_bag alias cone_node: reduced lidar max cone det distance 2.5 to 1.0 nav_node: adjusted cone detect distance from 45mm to 30mm so that it gets closer when touching rc.urdf: adjusted front tof sensors to more precisely detect the cone when real close.

File: urdfs/rc.urdf (robot description, URDF)
Before this commit: robot rc, 15 links, 14 joints
Joints:
- joint tof_fl_joint: origin xyz=-0.03 0.01 0.02 rpy=0.05 0 0.75 -> xyz=-0.02 0.01 0.02 rpy=0.05 0 0.75
- joint tof_fr_joint: origin xyz=0 -0.01 0.01 rpy=-0.05 0 -0.75 -> xyz=-0.02 -0.01 0.01 rpy=-0.05 0 -0.75

Commit message: rc.urdf: adjusted front tof z height and x rotation to place the ground reflection on the ground and remove tilt. adjusted lidar z rotation to align with tof using a cone really close to the bumber

File: urdfs/rc.urdf (robot description, URDF)
Before this commit: robot rc, 15 links, 14 joints
Joints:
- joint lidar_joint: origin xyz=0.180 0 0.300 rpy=0 0 -0.05 -> xyz=0.180 0 0.300 rpy=0 0 -0.02
- joint tof_fc_joint: origin xyz=0.650 0 0.09 rpy=0.0 -0.15 0.02 -> xyz=0.650 0 0.05 rpy=-0.05 -0.15 0.02

Commit message: rc.urdf: altered jeep body to have top and bottom. raised fron tof sensor to match rear sensor height and place in center of lower jeep section. Adjusted front tof sensor tilt to compensate for hiegher mount location

File: urdfs/rc.urdf (robot description, URDF)
Before this commit: robot rc, 15 links, 14 joints
Links:
- link base_link: geometry visual box size=0.480 0.380 0.100; visual box size=0.730 0.380 0.150
Joints:
- joint tof_fc_joint: origin xyz=0.650 0 0.05 rpy=-0.05 -0.15 0.02 -> xyz=0.650 0 0.120 rpy=-0.05 -0.10 0.02

Commit message: rc.urdf: Added L&R range sensors emulated with Lidar rc_params: Added range sensors to local map then commented out since they have same data as Lidar pcd_node: added range sensors using Lidar /scan topic data nav_node: added L&R range sensors to help driving manually obstacle detection. Used manual drive only for backup after touching cone, removed nav.backup use.

File: urdfs/rc.urdf (robot description, URDF)
Before this commit: robot rc, 15 links, 14 joints
Links:
- added link range_l_link; visual cylinder length=0.030 radius=0.020
- added link range_r_link; visual cylinder length=0.030 radius=0.020
Joints:
- added joint range_l_joint: type fixed, parent base_link, child range_l_link, origin xyz=0.180 0 0.300 rpy=0 0 1.571
- added joint range_r_joint: type fixed, parent base_link, child range_r_link, origin xyz=0.180 0 0.300 rpy=0 0 -1.571

Commit message: rc.urdf: Adjusted TOF fc, fr, fl rotations to have ground reflections level and at ground plane and verified that a box placed in front had a planar vertical surface with no seems between sensors

File: urdfs/rc.urdf (robot description, URDF)
Before this commit: robot rc, 17 links, 16 joints
Joints:
- joint tof_fc_joint: origin xyz=0.650 0 0.120 rpy=-0.05 -0.10 0.02 -> xyz=0.650 0 0.120 rpy=-0.05 -0.08 0.02
- joint tof_fl_joint: origin xyz=-0.02 0.01 0.02 rpy=0.05 0 0.75 -> xyz=-0.02 0.01 0.02 rpy=0.0 0.05 0.75
- joint tof_fr_joint: origin xyz=-0.02 -0.01 0.01 rpy=-0.05 0 -0.75 -> xyz=-0.02 -0.01 0.01 rpy=0.03 0.05 -0.75
